Commit message: Closer to actual robot.

File: urdf/my_robot.urdf (robot description, URDF)
Before this commit: robot my_robot, 5 links, 4 joints
Links:
- removed link caster_wheel
- added link front_caster, mass 0.5; collision sphere radius=0.03; visual sphere radius=0.03
- added link rear_caster, mass 0.5; collision sphere radius=0.03; visual sphere radius=0.03
- link base_link: mass 10.0 -> 6.8; geometry collision box size=0.305 0.305 0.254; visual box size=0.305 0.305 0.254
- link left_wheel: mass 0.5 -> 0.194; geometry collision cylinder length=0.032 radius=0.06; visual cylinder length=0.032 radius=0.06
- link right_wheel: mass 0.5 -> 0.194; geometry collision cylinder length=0.032 radius=0.06; visual cylinder length=0.032 radius=0.06
Joints:
- removed joint caster_joint
- added joint front_caster_joint: type fixed, parent base_link, child front_caster, origin xyz=0.12 0 -0.09
- added joint rear_caster_joint: type fixed, parent base_link, child rear_caster, origin xyz=-0.12 0 -0.09
- joint left_wheel_joint: axis 0 0 1 -> 0 1 0; origin xyz=0 0.1625 -0.06 rpy=1.5708 0 0 -> xyz=0 0.1685 -0.06
- joint lidar_joint: origin xyz=0 0 0.1 -> xyz=0 0 0.1905
- joint right_wheel_joint: axis 0 0 1 -> 0 1 0; origin xyz=0 -0.1625 -0.06 rpy=1.5708 0 0 -> xyz=0 -0.1685 -0.06
